File: Electronics/nokia-phone-arduino-shield/nokia-phone-arduino-shield.brd (EAGLE design)
At the start: 59.7 x 55.9 mm, 20 parts, among them J1 ARDUINO_R3_SHIELD, J3 ARDUINO_R3_SHIELD

Commit message: Routed and ready.
Parts:
- removed SJ21, SJ22: JUMPER-PAD-2-NC_BY_PASTE, SparkFun-Passives:PAD-JUMPER-2-NC_BY_PASTE_YES_SILK
- added JP4: (no value), SparkFun-Connectors:1X04_LOCK
- added JP5: (no value), SparkFun-Connectors:1X02_2.54_SCREWTERM
- added SJ1, SJ2: (no value), SparkFun-Retired:SJ_3
- moved JP3 3.81 mm to (38.1, 29.2)
Connections:
- removed net ARDUIN_TX: U2.12
- removed net FUBS_RX: POP6.P$1
- new net ARDUINO_TX: SJ2.2, U2.12
- net 5V: now also JP4.1, JP5.P2
- net ARDUINO_RX: now also SJ1.2
- net D13(SCK): now also SJ1.3
- net D5: now also SJ2.3
- net D8: now also SJ1.1; no longer SJ21.1, SJ21.2
- net D9: now also SJ2.1; no longer SJ22.1, SJ22.2
- net FBUS_RX: now also JP4.3, POP6.P$1
- net FBUS_TX: now also JP4.2
- net GND: now also JP4.4, JP5.P1
Routing:
- net 5V: track 5.33 -> 123.7 mm
- net FBUS_TX: track 0.00 -> 55.0 mm, vias 0 -> 3
- net FBUS_RX: track 0.00 -> 54.4 mm, vias 0 -> 1
- net D9: track 17.5 -> 59.1 mm, vias 2 -> 0
- net D8: track 17.0 -> 56.4 mm, vias 2 -> 0
- net D5: track 2.54 -> 41.0 mm
- net 3.3V: track 5.08 -> 40.9 mm, vias 1 -> 2
- net D13(SCK): track 2.79 -> 34.4 mm, vias 0 -> 2
- net ARDUINO_RX: track 0.00 -> 20.7 mm, vias 0 -> 2
- net ARDUINO_TX: track 0.00 -> 7.89 mm
Other:
- board text added: "100 nF"
- board text added: "FBusRX"
- board text added: "FBusTX"
- board text added: "Leo"
- board text added: "Leonardo"
- board text added: "RX"
- board text added: "Software serial"
- board text added: "TX"
- board text added: "Uno"
