File: Electronics/nokia-phone-arduino-shield/nokia-phone-arduino-shield.sch (EAGLE design)
At the start: 18 parts, among them J1 ARDUINO_R3_SHIELD, J3 ARDUINO_R3_SHIELD

Commit message: Routed and ready.
Parts:
- removed SJ21, SJ22: JUMPER-PAD-2-NC_BY_PASTE, SparkFun-Passives:JUMPER-PAD-2-NC_BY_PASTE
- added JP4: (no value), SparkFun-Connectors:M04LOCK
- added JP5: (no value), SparkFun-Connectors:M022.54MM_SCREWTERM
- added SJ1, SJ2: (no value), SparkFun-Retired:SOLDERJUMPER_2WAYS
Connections:
- removed net ARDUIN_TX: U2.B2
- removed net FUBS_RX: POP6.1
- new net ARDUINO_TX: SJ2.2, U2.B2
- net 5V: now also JP4.1, JP5.2
- net ARDUINO_RX: now also SJ1.2
- net D13(SCK): now also SJ1.3
- net D5: now also SJ2.3
- net D8: now also SJ1.1; no longer SJ21.1, SJ21.2
- net D9: now also SJ2.1; no longer SJ22.1, SJ22.2
- net FBUS_RX: now also JP4.3, POP6.1
- net FBUS_TX: now also JP4.2
- net GND: now also JP4.4, JP5.1
Other:
- note added: "F-Bus breakout"
- note added: "Leonardo"
- note added: "Nokia F-Bus cable"
- note added: "Uno"
- note removed: "USB connection"
Changed lines of the file:
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@@
 <part name="SUPPLY1" library="SparkFun-Aesthetics" deviceset="5V" device=""/>
 <part name="J3" library="SparkFun-Boards" deviceset="ARDUINO_R3_SHIELD" device="UNO_R3_SHIELD_NOLABELS_LOCK" value="ARDUINO_R3_SHIELD"/>
-<part name="SJ21" library="SparkFun-Passives" deviceset="JUMPER-PAD-2-NC_BY_PASTE" device=""/>
-<part name="SJ22" library="SparkFun-Passives" deviceset="JUMPER-PAD-2-NC_BY_PASTE" device=""/>
 <part name="GND2" library="SparkFun-Aesthetics" deviceset="GND" device=""/>
 <part name="P+2" library="SparkFun" deviceset="3.3V" device=""/>
@@
 <part name="GND11" library="SparkFun-Aesthetics" deviceset="GND" device=""/>
 <part name="SUPPLY9" library="SparkFun-Aesthetics" deviceset="5V" device=""/>
+<part name="SJ1" library="SparkFun-Retired" deviceset="SOLDERJUMPER_2WAY" device="S"/>
+<part name="SJ2" library="SparkFun-Retired" deviceset="SOLDERJUMPER_2WAY" device="S"/>
+<part name="JP4" library="SparkFun-Connectors" deviceset="M04" device="LOCK"/>
+<part name="SUPPLY10" library="SparkFun-Aesthetics" deviceset="5V" device=""/>
+<part name="GND12" library="SparkFun-Aesthetics" deviceset="GND" device=""/>
+<part name="JP5" library="SparkFun-Connectors" deviceset="M02" device="2.54MM_SCREWTERM"/>
+<part name="SUPPLY11" library="SparkFun-Aesthetics" deviceset="5V" device=""/>
+<part name="GND13" library="SparkFun-Aesthetics" deviceset="GND" device=""/>
 </parts>
 <sheets>
@@
 <wire x1="144.78" y1="190.5" x2="210.82" y2="190.5" width="0.2032" layer="94"/>
 <wire x1="210.82" y1="190.5" x2="210.82" y2="254" width="0.2032" layer="94"/>
-<text x="147.32" y="248.92" size="3.81" layer="94">USB connection</text>
+<text x="147.32" y="248.92" size="3.81" layer="94">Nokia F-Bus cable</text>
 <wire x1="144.78" y1="187.96" x2="144.78" y2="124.46" width="0.2032" layer="94"/>
 <wire x1="210.82" y1="187.96" x2="210.82" y2="124.46" width="0.2032" layer="94"/>
@@
 <wire x1="213.36" y1="190.5" x2="279.4" y2="190.5" width="0.2032" layer="94"/>
 <text x="215.9" y="248.92" size="3.81" layer="94">Power out</text>
+<text x="30.48" y="144.78" size="1.27" layer="97">Leonardo</text>
+<text x="30.48" y="172.72" size="1.27" layer="97">Uno</text>
+<wire x1="213.36" y1="187.96" x2="213.36" y2="124.46" width="0.2032" layer="94"/>
+<wire x1="213.36" y1="187.96" x2="279.4" y2="187.96" width="0.2032" layer="94"/>
+<wire x1="213.36" y1="124.46" x2="279.4" y2="124.46" width="0.2032" layer="94"/>
+<wire x1="279.4" y1="187.96" x2="279.4" y2="124.46" width="0.2032" layer="94"/>
+<text x="215.9" y="182.88" size="3.81" layer="94">F-Bus breakout</text>
 </plain>
 <instances>
@@
 <instance part="SUPPLY1" gate="G$1" x="17.78" y="213.36" rot="R90"/>
 <instance part="J3" gate="G$1" x="40.64" y="223.52"/>
-<instance part="SJ21" gate="G$1" x="15.24" y="177.8" smashed="yes"/>
-<instance part="SJ22" gate="G$1" x="15.24" y="172.72" smashed="yes"/>
 <instance part="GND2" gate="1" x="93.98" y="195.58"/>
 <instance part="P+2" gate="G$1" x="83.82" y="210.82" rot="R90"/>
@@
 <instance part="GND11" gate="1" x="238.76" y="203.2"/>
 <instance part="SUPPLY9" gate="G$1" x="238.76" y="213.36"/>
+<instance part="SJ1" gate="G$1" x="43.18" y="160.02"/>
+<instance part="SJ2" gate="G$1" x="45.72" y="157.48"/>
+<instance part="JP4" gate="G$1" x="236.22" y="167.64" rot="R180"/>
+<instance part="SUPPLY10" gate="G$1" x="228.6" y="172.72"/>
+<instance part="GND12" gate="1" x="228.6" y="157.48"/>
+<instance part="JP5" gate="G$1" x="248.92" y="208.28"/>
+<instance part="SUPPLY11" gate="G$1" x="259.08" y="213.36"/>
+<instance part="GND13" gate="1" x="259.08" y="203.2"/>
 </instances>
 <busses>
@@
 <wire x1="236.22" y1="208.28" x2="238.76" y2="208.28" width="0.1524" layer="91"/>
 </segment>
+<segment>
+<pinref part="JP4" gate="G$1" pin="4"/>
+<wire x1="231.14" y1="162.56" x2="228.6" y2="162.56" width="0.1524" layer="91"/>
+<pinref part="GND12" gate="1" pin="GND"/>
+<wire x1="228.6" y1="162.56" x2="228.6" y2="160.02" width="0.1524" layer="91"/>
+</segment>
+<segment>
+<pinref part="JP5" gate="G$1" pin="1"/>
+<wire x1="256.54" y1="208.28" x2="259.08" y2="208.28" width="0.1524" layer="91"/>
+<pinref part="GND13" gate="1" pin="GND"/>
+<wire x1="259.08" y1="205.74" x2="259.08" y2="208.28" width="0.1524" layer="91"/>
+</segment>
 </net>
 <net name="A1" class="0">
@@
 <label x="124.46" y="226.06" size="1.27" layer="95" xref="yes"/>
 <pinref part="J1" gate="G$1" pin="*D5"/>
+</segment>
+<segment>
+<pinref part="SJ2" gate="G$1" pin="3"/>
+<label x="35.56" y="149.86" size="1.27" layer="95" rot="R180" xref="yes"/>
+<wire x1="45.72" y1="152.4" x2="45.72" y2="149.86" width="0.1524" layer="91"/>
+<wire x1="45.72" y1="149.86" x2="35.56" y2="149.86" width="0.1524" layer="91"/>
 </segment>
 </net>
@@
 <wire x1="236.22" y1="210.82" x2="238.76" y2="210.82" width="0.1524" layer="91"/>
 </segment>
+<segment>
+<pinref part="SUPPLY10" gate="G$1" pin="5V"/>
+<pinref part="JP4" gate="G$1" pin="1"/>
+<wire x1="228.6" y1="172.72" x2="228.6" y2="170.18" width="0.1524" layer="91"/>
+<wire x1="228.6" y1="170.18" x2="231.14" y2="170.18" width="0.1524" layer="91"/>
+</segment>
+<segment>
+<pinref part="JP5" gate="G$1" pin="2"/>
+<wire x1="256.54" y1="210.82" x2="259.08" y2="210.82" width="0.1524" layer="91"/>
+<pinref part="SUPPLY11" gate="G$1" pin="5V"/>
+<wire x1="259.08" y1="210.82" x2="259.08" y2="213.36" width="0.1524" layer="91"/>
+</segment>
 </net>
 <net name="D3" class="0">
@@
 </segment>
 <segment>
-<pinref part="SJ21" gate="G$1" pin="2"/>
-<wire x1="20.32" y1="177.8" x2="20.32" y2="180.34" width="0.1524" layer="91"/>
-<pinref part="SJ21" gate="G$1" pin="1"/>
-<wire x1="20.32" y1="180.34" x2="10.16" y2="180.34" width="0.1524" layer="91"/>
-<wire x1="10.16" y1="180.34" x2="10.16" y2="177.8" width="0.1524" layer="91"/>
-<label x="20.32" y="177.8" size="1.27" layer="95" rot="MR180" xref="yes"/>
-</segment>
-<segment>
 <wire x1="124.46" y1="218.44" x2="121.92" y2="218.44" width="0.1524" layer="91"/>
 <label x="124.46" y="218.44" size="1.27" layer="95" xref="yes"/>
 <pinref part="J1" gate="G$1" pin="D8"/>
 </segment>
+<segment>
+<pinref part="SJ1" gate="G$1" pin="1"/>
+<label x="35.56" y="167.64" size="1.27" layer="95" rot="R180" xref="yes"/>
+<wire x1="43.18" y1="165.1" x2="43.18" y2="167.64" width="0.1524" layer="91"/>
+<wire x1="43.18" y1="167.64" x2="35.56" y2="167.64" width="0.1524" layer="91"/>
+</segment>
 </net>
 <net name="D9" class="0">
@@
 </segment>
 <segment>
-<pinref part="SJ22" gate="G$1" pin="2"/>
-<wire x1="20.32" y1="172.72" x2="20.32" y2="175.26" width="0.1524" layer="91"/>
-<pinref part="SJ22" gate="G$1" pin="1"/>
-<wire x1="20.32" y1="175.26" x2="10.16" y2="175.26" width="0.1524" layer="91"/>
-<wire x1="10.16" y1="175.26" x2="10.16" y2="172.72" width="0.1524" layer="91"/>
-<label x="20.32" y="172.72" size="1.27" layer="95" rot="MR180" xref="yes"/>
-</segment>
-<segment>
 <wire x1="124.46" y1="215.9" x2="121.92" y2="215.9" width="0.1524" layer="91"/>
 <label x="124.46" y="215.9" size="1.27" layer="95" xref="yes"/>
 <pinref part="J1" gate="G$1" pin="*D9"/>
 </segment>
+<segment>
+<pinref part="SJ2" gate="G$1" pin="1"/>
+<label x="35.56" y="170.18" size="1.27" layer="95" rot="R180" xref="yes"/>
+<wire x1="45.72" y1="162.56" x2="45.72" y2="170.18" width="0.1524" layer="91"/>
+<wire x1="45.72" y1="170.18" x2="35.56" y2="170.18" width="0.1524" layer="91"/>
+</segment>
 </net>
 <net name="D11(MOSI)" class="0">
@@
 <pinref part="J1" gate="G$1" pin="D13"/>
 </segment>
+<segment>
+<pinref part="SJ1" gate="G$1" pin="3"/>
+<label x="35.56" y="152.4" size="1.27" layer="95" rot="R180" xref="yes"/>
+<wire x1="43.18" y1="154.94" x2="43.18" y2="152.4" width="0.1524" layer="91"/>
+<wire x1="43.18" y1="152.4" x2="35.56" y2="152.4" width="0.1524" layer="91"/>
+</segment>
 </net>
 <net name="D6" class="0">
@@
 <label x="162.56" y="149.86" size="1.27" layer="95" rot="R180" xref="yes"/>
 </segment>
+<segment>
+<pinref part="JP4" gate="G$1" pin="2"/>
+<wire x1="231.14" y1="167.64" x2="228.6" y2="167.64" width="0.1524" layer="91"/>
+<label x="228.6" y="167.64" size="1.27" layer="95" rot="R180" xref="yes"/>
+</segment>
 </net>
 <net name="FBUS_RX" class="0">
@@
 <wire x1="91.44" y1="149.86" x2="93.98" y2="149.86" width="0.1524" layer="91"/>
 </segment>
-</net>
-<net name="FUBS_RX" class="0">
 <segment>
 <pinref part="POP6" gate="G$1" pin="1"/>
@@
 <label x="190.5" y="149.86" size="1.27" layer="95" xref="yes"/>
 </segment>
+<segment>
+<pinref part="JP4" gate="G$1" pin="3"/>
+<wire x1="231.14" y1="165.1" x2="228.6" y2="165.1" width="0.1524" layer="91"/>
+<label x="228.6" y="165.1" size="1.27" layer="95" rot="R180" xref="yes"/>
+</segment>
 </net>
 <net name="N$218" class="0">
@@
 <wire x1="127" y1="152.4" x2="124.46" y2="152.4" width="0.1524" layer="91"/>
 </segment>
-</net>
-<net name="ARDUIN_TX" class="0">
+<segment>
+<pinref part="SJ1" gate="G$1" pin="2"/>
+<wire x1="38.1" y1="160.02" x2="35.56" y2="160.02" width="0.1524" layer="91"/>
+<label x="35.56" y="160.02" size="1.27" layer="95" rot="R180" xref="yes"/>
+</segment>
+</net>
+<net name="ARDUINO_TX" class="0">
+<segment>
+<pinref part="SJ2" gate="G$1" pin="2"/>
+<wire x1="40.64" y1="157.48" x2="35.56" y2="157.48" width="0.1524" layer="91"/>
+<label x="35.56" y="157.48" size="1.27" layer="95" rot="R180" xref="yes"/>
+</segment>
 <segment>
 <label x="127" y="149.86" size="1.27" layer="95" xref="yes"/>
